Commit message: Update payload for simulated block_ft sensor.

File: urdf/gazebo_all_ft_demo.xacro (robot description, xacro)
@@ -103,5 +103,5 @@
     <parent link="block_ft_tool_mount" />
     <child link="m1100g" />
-    <origin xyz="0.03 0.05 0" rpy="0 0 0" />
+    <origin xyz="0.01 0.02 0.05" rpy="0 0 0" />
   </joint>
   <!-- Gazebo demo of the hex9904 sensor with 07mm hat and 73g payload. -->
